File: hardware/schematic/tat_v1/peripherals.kicad_sch (KiCad schematic)
At the start: 20 parts, among them SW3 SW_Push, SW4 SW_Push, SW5 SW_Push, U2 STS4x, U3 SHT4x, U4 BL24C08F, U5 ZD25Q128

Commit message: Simplified partslist and working on updated schematic
Parts:
- removed U5: ZD25Q128, symbol tat_library:ZD25Q128
Connections:
- net BTN_CENTER renamed Center Button
- net BTN_LEFT renamed Left Button
- net BTN_RIGHT renamed Right Button
- net EEPROM_SCL renamed EEPROM SCL
- net EEPROM_SDA renamed EEPROM SDA
- net SENSOR_SCL renamed Sensor SCL
- net SENSOR_SDA renamed Sensor SDA
- no-connect marks 2 -> 0
Other:
- note removed: "FLASH"
- moved on the sheet: C11, C12, C13, R10, R11, R12, R13, R14, R5, R6, R7, R8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

Commit message: Cleaned up basic schematic and double checked all components. Need to complete ERC.
Parts:
- added C19, C24: 100n, symbol Device:C_Small
- R11, R12, R13, R14: value 4k7 -> 10k
Connections:
- net +3.3V: now also C19.1, C24.1
- net GND: now also C19.2, C24.2
Other:
- note added: "Debouncing circuit taken from How to implement Hardware debounce for switches and relays by Digikey Schmitt trigger omitted for simplicity since STM32 has one built in Diode omitted since we only care about switch activation"
- note added: "EEPROM I2C address varies with byte address, see datasheet for details"
- note added: "Temperature & humidity sensors"
- note added: "User inputs"
- note removed: "Double check pull up resistor values!"
- note removed: "TEMP & HUMIDITY SENSORS"
- note removed: "User Inputs"
- moved on the sheet: U3

Commit message: Added new titles to sheets
Other:
- title: (none) -> Tiny Ambient Tracker - peripherals & user input
Changed lines of the file:
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@@
 	(generator_version "9.0")
 	(paper "A4")
+	(title_block
+		(title "Tiny Ambient Tracker - peripherals & user input")
+	)
 	(text "Temperature & humidity\nsensors"
 		(exclude_from_sim no)

Commit message: Used auto reference designator on whole schematic
Parts:
- renumbered C11 to C19, C12 to C20, C13 to C21, C19 to C22, C24 to C23, R6 to R18, R8 to R19, R10 to R20, R5 to R21, R7 to R22, R9 to R23, R11 to R24, R12 to R25, R13 to R26, R14 to R27, SW3 to SW4, SW4 to SW5, SW5 to SW6, U2 to U5, U3 to U6, U4 to U7

Commit message: Continuing with setting basic footprints for parts
Parts:
- C18: renamed from C19; footprint (none) -> Capacitor_SMD:C_0402_1005Metric
- C19: renamed from C20; footprint (none) -> Capacitor_SMD:C_0402_1005Metric
- C20: renamed from C21; footprint (none) -> Capacitor_SMD:C_0402_1005Metric
- C21: renamed from C22; footprint (none) -> Capacitor_SMD:C_0402_1005Metric
- C22: renamed from C23; footprint (none) -> Capacitor_SMD:C_0402_1005Metric
- R18, R19, R20, R21, R22, R23, R24, R25, R26, R27: footprint (none) -> Resistor_SMD:R_0402_1005Metric
Changed lines of the file:
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@@
 		(on_board yes)
 		(dnp no)
-		(property "Reference" "#PWR044"
+		(property "Reference" "#PWR043"
 			(at 161.29 77.47 0)
 			(effects
@@
 			(project "tat_v1"
 				(path "/b6d2ddf1-6792-45dd-afc9-29fd74d587ec/c7fedf3e-0076-4d27-8f18-2fdc24044d55"
-					(reference "#PWR044")
+					(reference "#PWR043")
 					(unit 1)
 				)
@@
 		(on_board yes)
 		(dnp no)
-		(property "Reference" "#PWR048"
+		(property "Reference" "#PWR047"
 			(at 228.6 85.09 0)
 			(effects
@@
 			(project "tat_v1"
 				(path "/b6d2ddf1-6792-45dd-afc9-29fd74d587ec/c7fedf3e-0076-4d27-8f18-2fdc24044d55"
-					(reference "#PWR048")
+					(reference "#PWR047")
 					(unit 1)
 				)
@@
 			)
 		)
-		(property "Footprint" ""
+		(property "Footprint" "Resistor_SMD:R_0402_1005Metric"
 			(at 141.732 83.82 90)
 			(effects
@@
 			)
 		)
-		(property "Footprint" ""
+		(property "Footprint" "Resistor_SMD:R_0402_1005Metric"
 			(at 57.15 98.298 90)
 			(effects
@@
 		(dnp no)
 		(fields_autoplaced yes)
-		(property "Reference" "C20"
+		(property "Reference" "C19"
 			(at 67.31 104.1462 0)
 			(effects
@@
 			)
 		)
-		(property "Footprint" ""
+		(property "Footprint" "Capacitor_SMD:C_0402_1005Metric"
 			(at 64.77 105.41 0)
 			(effects
@@
 			(project "tat_v1"
 				(path "/b6d2ddf1-6792-45dd-afc9-29fd74d587ec/c7fedf3e-0076-4d27-8f18-2fdc24044d55"
-					(reference "C20")
+					(reference "C19")
 					(unit 1)
 				)
@@
 		(on_board yes)
 		(dnp no)
-		(property "Reference" "C23"
+		(property "Reference" "C22"
 			(at 170.18 112.776 90)
 			(effects
@@
 			)
 		)
-		(property "Footprint" ""
+		(property "Footprint" "Capacitor_SMD:C_0402_1005Metric"
 			(at 170.18 115.57 0)
 			(effects
@@
 			(project "tat_v1"
 				(path "/b6d2ddf1-6792-45dd-afc9-29fd74d587ec/c7fedf3e-0076-4d27-8f18-2fdc24044d55"
-					(reference "C23")
+					(reference "C22")
 					(unit 1)
 				)
@@
 			)
 		)
-		(property "Footprint" ""
+		(property "Footprint" "Resistor_SMD:R_0402_1005Metric"
 			(at 62.992 132.08 90)
 			(effects
@@
 		(on_board yes)
 		(dnp no)
-		(property "Reference" "C22"
+		(property "Reference" "C21"
 			(at 170.18 75.946 90)
 			(effects
@@
 			)
 		)
-		(property "Footprint" ""
+		(property "Footprint" "Capacitor_SMD:C_0402_1005Metric"
 			(at 170.18 78.74 0)
 			(effects
@@
 			(project "tat_v1"
 				(path "/b6d2ddf1-6792-45dd-afc9-29fd74d587ec/c7fedf3e-0076-4d27-8f18-2fdc24044d55"
-					(reference "C22")
+					(reference "C21")
 					(unit 1)
 				)
@@
 		(on_board yes)
 		(dnp no)
-		(property "Reference" "#PWR042"
+		(property "Reference" "#PWR041"
 			(at 64.77 90.17 0)
 			(effects
@@
 			(project "tat_v1"
 				(path "/b6d2ddf1-6792-45dd-afc9-29fd74d587ec/c7fedf3e-0076-4d27-8f18-2fdc24044d55"
-					(reference "#PWR042")
+					(reference "#PWR041")
 					(unit 1)
 				)
@@
 		(dnp no)
 		(fields_autoplaced yes)
-		(property "Reference" "#PWR039"
+		(property "Reference" "#PWR038"
 			(at 58.42 121.92 0)
 			(effects
@@
 			(project "tat_v1"
 				(path "/b6d2ddf1-6792-45dd-afc9-29fd74d587ec/c7fedf3e-0076-4d27-8f18-2fdc24044d55"
-					(reference "#PWR039")
+					(reference "#PWR038")
 					(unit 1)
 				)
@@
 		(dnp no)
 		(fields_autoplaced yes)
-		(property "Reference" "#PWR045"
+		(property "Reference" "#PWR044"
 			(at 161.29 109.22 0)
 			(effects
@@
 			(project "tat_v1"
 				(path "/b6d2ddf1-6792-45dd-afc9-29fd74d587ec/c7fedf3e-0076-4d27-8f18-2fdc24044d55"
-					(reference "#PWR045")
+					(reference "#PWR044")
 					(unit 1)
 				)
@@
 			)
 		)
-		(property "Footprint" ""
+		(property "Footprint" "Resistor_SMD:R_0402_1005Metric"
 			(at 57.15 138.938 90)
 			(effects
@@
 		(dnp no)
 		(fields_autoplaced yes)
-		(property "Reference" "#PWR040"
+		(property "Reference" "#PWR039"
 			(at 58.42 162.56 0)
 			(effects
@@
 			(project "tat_v1"
 				(path "/b6d2ddf1-6792-45dd-afc9-29fd74d587ec/c7fedf3e-0076-4d27-8f18-2fdc24044d55"
-					(reference "#PWR040")
+					(reference "#PWR039")
 					(unit 1)
 				)
@@
 		(on_board yes)
 		(dnp no)
-		(property "Reference" "#PWR041"
+		(property "Reference" "#PWR040"
 			(at 64.77 50.8 0)
 			(effects
@@
 			(project "tat_v1"
 				(path "/b6d2ddf1-6792-45dd-afc9-29fd74d587ec/c7fedf3e-0076-4d27-8f18-2fdc24044d55"
-					(reference "#PWR041")
+					(reference "#PWR040")
 					(unit 1)
 				)
@@
 		(on_board yes)
 		(dnp no)
-		(property "Reference" "#PWR043"
+		(property "Reference" "#PWR042"
 			(at 64.77 130.81 0)
 			(effects
@@
 			(project "tat_v1"
 				(path "/b6d2ddf1-6792-45dd-afc9-29fd74d587ec/c7fedf3e-0076-4d27-8f18-2fdc24044d55"
-					(reference "#PWR043")
+					(reference "#PWR042")
 					(unit 1)
 				)
@@
 		(dnp no)
 		(fields_autoplaced yes)
-		(property "Reference" "#PWR049"
+		(property "Reference" "#PWR048"
 			(at 228.6 116.84 0)
 			(effects
@@
 			(project "tat_v1"
 				(path "/b6d2ddf1-6792-45dd-afc9-29fd74d587ec/c7fedf3e-0076-4d27-8f18-2fdc24044d55"
-					(reference "#PWR049")
+					(reference "#PWR048")
 					(unit 1)
 				)
@@
 		(dnp no)
 		(fields_autoplaced yes)
-		(property "Reference" "C21"
+		(property "Reference" "C20"
 			(at 67.31 144.7862 0)
 			(effects
@@
 			)
 		)
-		(property "Footprint" ""
+		(property "Footprint" "Capacitor_SMD:C_0402_1005Metric"
 			(at 64.77 146.05 0)
 			(effects
@@
 			(project "tat_v1"
 				(path "/b6d2ddf1-6792-45dd-afc9-29fd74d587ec/c7fedf3e-0076-4d27-8f18-2fdc24044d55"
-					(reference "C21")
+					(reference "C20")
 					(unit 1)
 				)
@@
 			)
 		)
-		(property "Footprint" ""
+		(property "Footprint" "Resistor_SMD:R_0402_1005Metric"
 			(at 240.792 90.17 90)
 			(effects
@@
 		(dnp no)
 		(fields_autoplaced yes)
-		(property "Reference" "C19"
+		(property "Reference" "C18"
 			(at 67.31 64.7762 0)
 			(effects
@@
 			)
 		)
-		(property "Footprint" ""
+		(property "Footprint" "Capacitor_SMD:C_0402_1005Metric"
 			(at 64.77 66.04 0)
 			(effects
@@
 			(project "tat_v1"
 				(path "/b6d2ddf1-6792-45dd-afc9-29fd74d587ec/c7fedf3e-0076-4d27-8f18-2fdc24044d55"
-					(reference "C19")
+					(reference "C18")
 					(unit 1)
 				)
@@
 		(dnp no)
 		(fields_autoplaced yes)
-		(property "Reference" "#PWR047"
+		(property "Reference" "#PWR046"
 			(at 161.29 144.78 0)
 			(effects
@@
 			(project "tat_v1"
 				(path "/b6d2ddf1-6792-45dd-afc9-29fd74d587ec/c7fedf3e-0076-4d27-8f18-2fdc24044d55"
-					(reference "#PWR047")
+					(reference "#PWR046")
 					(unit 1)
 				)
@@
 			)
 		)
-		(property "Footprint" ""
+		(property "Footprint" "Resistor_SMD:R_0402_1005Metric"
 			(at 249.682 90.17 90)
 			(effects
@@
 		(dnp no)
 		(fields_autoplaced yes)
-		(property "Reference" "#PWR038"
+		(property "Reference" "#PWR037"
 			(at 58.42 82.55 0)
 			(effects
@@
 			(project "tat_v1"
 				(path "/b6d2ddf1-6792-45dd-afc9-29fd74d587ec/c7fedf3e-0076-4d27-8f18-2fdc24044d55"
-					(reference "#PWR038")
+					(reference "#PWR037")
 					(unit 1)
 				)
@@
 		(on_board yes)
 		(dnp no)
-		(property "Reference" "#PWR046"
+		(property "Reference" "#PWR045"
 			(at 161.29 118.11 0)
 			(effects
@@
 			(project "tat_v1"
 				(path "/b6d2ddf1-6792-45dd-afc9-29fd74d587ec/c7fedf3e-0076-4d27-8f18-2fdc24044d55"
-					(reference "#PWR046")
+					(reference "#PWR045")
 					(unit 1)
 				)
@@
 			)
 		)
-		(property "Footprint" ""
+		(property "Footprint" "Resistor_SMD:R_0402_1005Metric"
 			(at 132.842 83.82 90)
 			(effects
@@
 			)
 		)
-		(property "Footprint" ""
+		(property "Footprint" "Resistor_SMD:R_0402_1005Metric"
 			(at 57.15 58.928 90)
 			(effects
@@
 			)
 		)
-		(property "Footprint" ""
+		(property "Footprint" "Resistor_SMD:R_0402_1005Metric"
 			(at 62.992 52.07 90)
 			(effects
@@
 			)
 		)
-		(property "Footprint" ""
+		(property "Footprint" "Resistor_SMD:R_0402_1005Metric"
 			(at 62.992 91.44 90)
 			(effects

Commit message: Continuing work on setting parts footprints
Parts:
- R21, R22, R23, R24, R25, R26, R27: Link (none) -> https://www.lcsc.com/product-detail/Chip-Resistor-Surface-M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
Changed lines of the file:
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@@
 			)
 		)
-		(property "Datasheet" "~"
+		(property "Datasheet" "https://www.lcsc.com/datasheet/lcsc_datasheet_2411221126_UNI-ROYAL-Uniroyal-Elec-0402WGF1002TCE_C25744.pdf"
 			(at 143.51 83.82 0)
 			(effects
@@
 		)
 		(property "Description" "Resistor"
+			(at 143.51 83.82 0)
+			(effects
+				(font
+					(size 1.27 1.27)
+				)
+				(hide yes)
+			)
+		)
+		(property "Link" "https://www.lcsc.com/product-detail/Chip-Resistor-Surface-Mount_UNI-ROYAL-Uniroyal-Elec-0402WGF1002TCE_C25744.html"
 			(at 143.51 83.82 0)
 			(effects
@@
 			)
 		)
-		(property "Datasheet" "~"
+		(property "Datasheet" "https://www.lcsc.com/datasheet/lcsc_datasheet_2411221126_UNI-ROYAL-Uniroyal-Elec-0402WGF1002TCE_C25744.pdf"
 			(at 64.77 132.08 0)
 			(effects
@@
 		)
 		(property "Description" "Resistor"
+			(at 64.77 132.08 0)
+			(effects
+				(font
+					(size 1.27 1.27)
+				)
+				(hide yes)
+			)
+		)
+		(property "Link" "https://www.lcsc.com/product-detail/Chip-Resistor-Surface-Mount_UNI-ROYAL-Uniroyal-Elec-0402WGF1002TCE_C25744.html"
 			(at 64.77 132.08 0)
 			(effects
@@
 			)
 		)
-		(property "Datasheet" "~"
+		(property "Datasheet" "https://www.lcsc.com/datasheet/lcsc_datasheet_2411221126_UNI-ROYAL-Uniroyal-Elec-0402WGF1002TCE_C25744.pdf"
 			(at 242.57 90.17 0)
 			(effects
@@
 		)
 		(property "Description" "Resistor"
+			(at 242.57 90.17 0)
+			(effects
+				(font
+					(size 1.27 1.27)
+				)
+				(hide yes)
+			)
+		)
+		(property "Link" "https://www.lcsc.com/product-detail/Chip-Resistor-Surface-Mount_UNI-ROYAL-Uniroyal-Elec-0402WGF1002TCE_C25744.html"
 			(at 242.57 90.17 0)
 			(effects
@@
 			)
 		)
-		(property "Datasheet" "~"
+		(property "Datasheet" "https://www.lcsc.com/datasheet/lcsc_datasheet_2411221126_UNI-ROYAL-Uniroyal-Elec-0402WGF1002TCE_C25744.pdf"
 			(at 251.46 90.17 0)
 			(effects
@@
 		)
 		(property "Description" "Resistor"
+			(at 251.46 90.17 0)
+			(effects
+				(font
+					(size 1.27 1.27)
+				)
+				(hide yes)
+			)
+		)
+		(property "Link" "https://www.lcsc.com/product-detail/Chip-Resistor-Surface-Mount_UNI-ROYAL-Uniroyal-Elec-0402WGF1002TCE_C25744.html"
 			(at 251.46 90.17 0)
 			(effects
@@
 			)
 		)
-		(property "Datasheet" "~"
+		(property "Datasheet" "https://www.lcsc.com/datasheet/lcsc_datasheet_2411221126_UNI-ROYAL-Uniroyal-Elec-0402WGF1002TCE_C25744.pdf"
 			(at 134.62 83.82 0)
 			(effects
@@
 		)
 		(property "Description" "Resistor"
+			(at 134.62 83.82 0)
+			(effects
+				(font
+					(size 1.27 1.27)
+				)
+				(hide yes)
+			)
+		)
+		(property "Link" "https://www.lcsc.com/product-detail/Chip-Resistor-Surface-Mount_UNI-ROYAL-Uniroyal-Elec-0402WGF1002TCE_C25744.html"
 			(at 134.62 83.82 0)
 			(effects
@@
 			)
 		)
-		(property "Datasheet" "~"
+		(property "Datasheet" "https://www.lcsc.com/datasheet/lcsc_datasheet_2411221126_UNI-ROYAL-Uniroyal-Elec-0402WGF1002TCE_C25744.pdf"
 			(at 64.77 52.07 0)
 			(effects
@@
 		)
 		(property "Description" "Resistor"
+			(at 64.77 52.07 0)
+			(effects
+				(font
+					(size 1.27 1.27)
+				)
+				(hide yes)
+			)
+		)
+		(property "Link" "https://www.lcsc.com/product-detail/Chip-Resistor-Surface-Mount_UNI-ROYAL-Uniroyal-Elec-0402WGF1002TCE_C25744.html"
 			(at 64.77 52.07 0)
 			(effects
@@
 			)
 		)
-		(property "Datasheet" "~"
+		(property "Datasheet" "https://www.lcsc.com/datasheet/lcsc_datasheet_2411221126_UNI-ROYAL-Uniroyal-Elec-0402WGF1002TCE_C25744.pdf"
 			(at 64.77 91.44 0)
 			(effects
@@
 			(at 64.77 91.44 0)
 			(effects
+				(font
+					(size 1.27 1.27)
+				)
+				(hide yes)
+			)
+		)
+		(property "Link" "https://www.lcsc.com/product-detail/Chip-Resistor-Surface-Mount_UNI-ROYAL-Uniroyal-Elec-0402WGF1002TCE_C25744.html"
+			(at 64.77 91.44 0)
+			(effects
