File: hardware/schematic/tat_v1/peripherals.kicad_sch (KiCad schematic)
At the start: 21 parts, among them SW4 SW_Push, SW5 SW_Push, SW6 SW_Push, U5 STS4x, U6 SHT4x, U7 BL24C08F

Commit message: Most simple footprints added. Need to create footprints for more complex parts.
Parts:
- C19: renamed from C18; Link (none) -> https://www.lcsc.com/product-detail/Multilayer-Ceramic-Capa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
- C20: renamed from C19; Link (none) -> https://www.lcsc.com/product-detail/Multilayer-Ceramic-Capa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
- C21: renamed from C20; Link (none) -> https://www.lcsc.com/product-detail/Multilayer-Ceramic-Capa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
- C22: renamed from C21; Link (none) -> https://www.lcsc.com/product-detail/Multilayer-Ceramic-Capa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
- C23: renamed from C22; Link (none) -> https://www.lcsc.com/product-detail/Multilayer-Ceramic-Capa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
- SW4: Link (none) -> https://www.lcsc.com/product-detail/Tactile-Switches_SHOU-H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
Changed lines of the file:
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@@
 		(on_board yes)
 		(dnp no)
-		(property "Reference" "#PWR043"
+		(property "Reference" "#PWR044"
 			(at 161.29 77.47 0)
 			(effects
@@
 			(project "tat_v1"
 				(path "/b6d2ddf1-6792-45dd-afc9-29fd74d587ec/c7fedf3e-0076-4d27-8f18-2fdc24044d55"
-					(reference "#PWR043")
+					(reference "#PWR044")
 					(unit 1)
 				)
@@
 		(on_board yes)
 		(dnp no)
-		(property "Reference" "#PWR047"
+		(property "Reference" "#PWR048"
 			(at 228.6 85.09 0)
 			(effects
@@
 			(project "tat_v1"
 				(path "/b6d2ddf1-6792-45dd-afc9-29fd74d587ec/c7fedf3e-0076-4d27-8f18-2fdc24044d55"
-					(reference "#PWR047")
+					(reference "#PWR048")
 					(unit 1)
 				)
@@
 			)
 		)
-		(property "Datasheet" "~"
+		(property "Datasheet" "https://www.lcsc.com/datasheet/lcsc_datasheet_2404241539_SHOU-HAN-TS24CA_C393942.pdf"
 			(at 46.99 66.04 0)
 			(effects
@@
 			)
 		)
+		(property "Link" "https://www.lcsc.com/product-detail/Tactile-Switches_SHOU-HAN-TS24CA_C393942.html?s_z=n_SHOU%2520HAN%2520TS24CA"
+			(at 52.07 66.04 90)
+			(effects
+				(font
+					(size 1.27 1.27)
+				)
+				(hide yes)
+			)
+		)
 		(pin "2"
 		)
@@
 		(dnp no)
 		(fields_autoplaced yes)
-		(property "Reference" "C19"
+		(property "Reference" "C20"
 			(at 67.31 104.1462 0)
 			(effects
@@
 			)
 		)
-		(property "Datasheet" "~"
+		(property "Datasheet" "https://www.lcsc.com/datasheet/lcsc_datasheet_2203221430_YAGEO-CC0402KRX7R7BB104_C60474.pdf"
 			(at 64.77 105.41 0)
 			(effects
@@
 			)
 		)
+		(property "Link" "https://www.lcsc.com/product-detail/Multilayer-Ceramic-Capacitors-MLCC-SMD-SMT_YAGEO-CC0402KRX7R7BB104_C60474.html"
+			(at 64.77 105.41 0)
+			(effects
+				(font
+					(size 1.27 1.27)
+				)
+				(hide yes)
+			)
+		)
 		(pin "1"
 		)
@@
 			(project "tat_v1"
 				(path "/b6d2ddf1-6792-45dd-afc9-29fd74d587ec/c7fedf3e-0076-4d27-8f18-2fdc24044d55"
-					(reference "C19")
+					(reference "C20")
 					(unit 1)
 				)
@@
 		(on_board yes)
 		(dnp no)
-		(property "Reference" "C22"
+		(property "Reference" "C23"
 			(at 170.18 112.776 90)
 			(effects
@@
 			)
 		)
-		(property "Datasheet" "~"
+		(property "Datasheet" "https://www.lcsc.com/datasheet/lcsc_datasheet_2203221430_YAGEO-CC0402KRX7R7BB104_C60474.pdf"
 			(at 170.18 115.57 0)
 			(effects
@@
 			)
 		)
+		(property "Link" "https://www.lcsc.com/product-detail/Multilayer-Ceramic-Capacitors-MLCC-SMD-SMT_YAGEO-CC0402KRX7R7BB104_C60474.html"
+			(at 170.18 115.57 90)
+			(effects
+				(font
+					(size 1.27 1.27)
+				)
+				(hide yes)
+			)
+		)
 		(pin "1"
 		)
@@
 			(project "tat_v1"
 				(path "/b6d2ddf1-6792-45dd-afc9-29fd74d587ec/c7fedf3e-0076-4d27-8f18-2fdc24044d55"
-					(reference "C22")
+					(reference "C23")
 					(unit 1)
 				)
@@
 		(on_board yes)
 		(dnp no)
-		(property "Reference" "C21"
+		(property "Reference" "C22"
 			(at 170.18 75.946 90)
 			(effects
@@
 			)
 		)
-		(property "Datasheet" "~"
+		(property "Datasheet" "https://www.lcsc.com/datasheet/lcsc_datasheet_2203221430_YAGEO-CC0402KRX7R7BB104_C60474.pdf"
 			(at 170.18 78.74 0)
 			(effects
@@
 			)
 		)
+		(property "Link" "https://www.lcsc.com/product-detail/Multilayer-Ceramic-Capacitors-MLCC-SMD-SMT_YAGEO-CC0402KRX7R7BB104_C60474.html"
+			(at 170.18 78.74 90)
+			(effects
+				(font
+					(size 1.27 1.27)
+				)
+				(hide yes)
+			)
+		)
 		(pin "1"
 		)
@@
 			(project "tat_v1"
 				(path "/b6d2ddf1-6792-45dd-afc9-29fd74d587ec/c7fedf3e-0076-4d27-8f18-2fdc24044d55"
-					(reference "C21")
+					(reference "C22")
 					(unit 1)
 				)
@@
 		(on_board yes)
 		(dnp no)
-		(property "Reference" "#PWR041"
+		(property "Reference" "#PWR042"
 			(at 64.77 90.17 0)
 			(effects
@@
 			(project "tat_v1"
 				(path "/b6d2ddf1-6792-45dd-afc9-29fd74d587ec/c7fedf3e-0076-4d27-8f18-2fdc24044d55"
-					(reference "#PWR041")
+					(reference "#PWR042")
 					(unit 1)
 				)
@@
 		(dnp no)
 		(fields_autoplaced yes)
-		(property "Reference" "#PWR038"
+		(property "Reference" "#PWR039"
 			(at 58.42 121.92 0)
 			(effects
@@
 			(project "tat_v1"
 				(path "/b6d2ddf1-6792-45dd-afc9-29fd74d587ec/c7fedf3e-0076-4d27-8f18-2fdc24044d55"
-					(reference "#PWR038")
+					(reference "#PWR039")
 					(unit 1)
 				)
@@
 		(dnp no)
 		(fields_autoplaced yes)
-		(property "Reference" "#PWR044"
+		(property "Reference" "#PWR045"
 			(at 161.29 109.22 0)
 			(effects
@@
 			(project "tat_v1"
 				(path "/b6d2ddf1-6792-45dd-afc9-29fd74d587ec/c7fedf3e-0076-4d27-8f18-2fdc24044d55"
-					(reference "#PWR044")
+					(reference "#PWR045")
 					(unit 1)
 				)
@@
 		(dnp no)
 		(fields_autoplaced yes)
-		(property "Reference" "#PWR039"
+		(property "Reference" "#PWR040"
 			(at 58.42 162.56 0)
 			(effects
@@
 			(project "tat_v1"
 				(path "/b6d2ddf1-6792-45dd-afc9-29fd74d587ec/c7fedf3e-0076-4d27-8f18-2fdc24044d55"
-					(reference "#PWR039")
+					(reference "#PWR040")
 					(unit 1)
 				)
@@
 		(on_board yes)
 		(dnp no)
-		(property "Reference" "#PWR040"
+		(property "Reference" "#PWR041"
 			(at 64.77 50.8 0)
 			(effects
@@
 			(project "tat_v1"
 				(path "/b6d2ddf1-6792-45dd-afc9-29fd74d587ec/c7fedf3e-0076-4d27-8f18-2fdc24044d55"
-					(reference "#PWR040")
+					(reference "#PWR041")
 					(unit 1)
 				)
@@
 		(on_board yes)
 		(dnp no)
-		(property "Reference" "#PWR042"
+		(property "Reference" "#PWR043"
 			(at 64.77 130.81 0)
 			(effects
@@
 			(project "tat_v1"
 				(path "/b6d2ddf1-6792-45dd-afc9-29fd74d587ec/c7fedf3e-0076-4d27-8f18-2fdc24044d55"
-					(reference "#PWR042")
+					(reference "#PWR043")
 					(unit 1)
 				)
@@
 		(dnp no)
 		(fields_autoplaced yes)
-		(property "Reference" "#PWR048"
+		(property "Reference" "#PWR049"
 			(at 228.6 116.84 0)
 			(effects
@@
 			(project "tat_v1"
 				(path "/b6d2ddf1-6792-45dd-afc9-29fd74d587ec/c7fedf3e-0076-4d27-8f18-2fdc24044d55"
-					(reference "#PWR048")
+					(reference "#PWR049")
 					(unit 1)
 				)
@@
 		(dnp no)
 		(fields_autoplaced yes)
-		(property "Reference" "C20"
+		(property "Reference" "C21"
 			(at 67.31 144.7862 0)
 			(effects
@@
 			)
 		)
-		(property "Datasheet" "~"
+		(property "Datasheet" "https://www.lcsc.com/datasheet/lcsc_datasheet_2203221430_YAGEO-CC0402KRX7R7BB104_C60474.pdf"
 			(at 64.77 146.05 0)
 			(effects
@@
 			)
 		)
+		(property "Link" "https://www.lcsc.com/product-detail/Multilayer-Ceramic-Capacitors-MLCC-SMD-SMT_YAGEO-CC0402KRX7R7BB104_C60474.html"
+			(at 64.77 146.05 0)
+			(effects
+				(font
+					(size 1.27 1.27)
+				)
+				(hide yes)
+			)
+		)
 		(pin "1"
 		)
@@
 			(project "tat_v1"
 				(path "/b6d2ddf1-6792-45dd-afc9-29fd74d587ec/c7fedf3e-0076-4d27-8f18-2fdc24044d55"
-					(reference "C20")
+					(reference "C21")
 					(unit 1)
 				)
@@
 		(dnp no)
 		(fields_autoplaced yes)
-		(property "Reference" "C18"
+		(property "Reference" "C19"
 			(at 67.31 64.7762 0)
 			(effects
@@
 			)
 		)
-		(property "Datasheet" "~"
+		(property "Datasheet" "https://www.lcsc.com/datasheet/lcsc_datasheet_2203221430_YAGEO-CC0402KRX7R7BB104_C60474.pdf"
 			(at 64.77 66.04 0)
 			(effects
@@
 			)
 		)
+		(property "Link" "https://www.lcsc.com/product-detail/Multilayer-Ceramic-Capacitors-MLCC-SMD-SMT_YAGEO-CC0402KRX7R7BB104_C60474.html"
+			(at 64.77 66.04 0)
+			(effects
+				(font
+					(size 1.27 1.27)
+				)
+				(hide yes)
+			)
+		)
 		(pin "1"
 		)
@@
 			(project "tat_v1"
 				(path "/b6d2ddf1-6792-45dd-afc9-29fd74d587ec/c7fedf3e-0076-4d27-8f18-2fdc24044d55"
-					(reference "C18")
+					(reference "C19")
 					(unit 1)
 				)
@@
 		(dnp no)
 		(fields_autoplaced yes)
-		(property "Reference" "#PWR046"
+		(property "Reference" "#PWR047"
 			(at 161.29 144.78 0)
 			(effects
@@
 			(project "tat_v1"
 				(path "/b6d2ddf1-6792-45dd-afc9-29fd74d587ec/c7fedf3e-0076-4d27-8f18-2fdc24044d55"
-					(reference "#PWR046")
+					(reference "#PWR047")
 					(unit 1)
 				)
@@
 		(dnp no)
 		(fields_autoplaced yes)
-		(property "Reference" "#PWR037"
+		(property "Reference" "#PWR038"
 			(at 58.42 82.55 0)
 			(effects
@@
 			(project "tat_v1"
 				(path "/b6d2ddf1-6792-45dd-afc9-29fd74d587ec/c7fedf3e-0076-4d27-8f18-2fdc24044d55"
-					(reference "#PWR037")
+					(reference "#PWR038")
 					(unit 1)
 				)
@@
 		(on_board yes)
 		(dnp no)
-		(property "Reference" "#PWR045"
+		(property "Reference" "#PWR046"
 			(at 161.29 118.11 0)
 			(effects
@@
 			(project "tat_v1"
 				(path "/b6d2ddf1-6792-45dd-afc9-29fd74d587ec/c7fedf3e-0076-4d27-8f18-2fdc24044d55"
-					(reference "#PWR045")
-					(unit 1)
-				)
+					(reference "#PWR046")
+					(unit 1)
+				)

Commit message: Finished all footprints, can now start laying out circuit
Parts:
- SW4, SW5, SW6: value SW_Push -> SW_Push_RightAngle; footprint (none) -> tat_footprints:SW_Push_SHOU_HAN_SPST_RightAngle_TS24CA
- U5, U6: footprint (none) -> Sensor_Humidity:Sensirion_DFN-4_1.5x1.5mm_P0.8mm_SHT4x_NoCentralPad
- U7: footprint (none) -> Package_DFN_QFN:DFN-8-1EP_3x2mm_P0.5mm_EP1.3x1.5mm
- renumbered R18 to R21, R19 to R22, R20 to R23, R21 to R24, R22 to R25, R23 to R26, R24 to R27, R25 to R28, R26 to R29, R27 to R30
Changed lines of the file:
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@@
 		(dnp no)
 		(fields_autoplaced yes)
-		(property "Reference" "R25"
+		(property "Reference" "R28"
 			(at 146.05 82.5499 0)
 			(effects
@@
 			(project "tat_v1"
 				(path "/b6d2ddf1-6792-45dd-afc9-29fd74d587ec/c7fedf3e-0076-4d27-8f18-2fdc24044d55"
-					(reference "R25")
+					(reference "R28")
 					(unit 1)
 				)
@@
 			)
 		)
-		(property "Footprint" ""
+		(property "Footprint" "Package_DFN_QFN:DFN-8-1EP_3x2mm_P0.5mm_EP1.3x1.5mm"
 			(at 228.6 99.06 0)
 			(effects
@@
 		(dnp no)
 		(property "Reference" "SW5"
-			(at 43.688 103.886 90)
-			(effects
-				(font
-					(size 1.27 1.27)
-				)
-			)
-		)
-		(property "Value" "SW_Push"
-			(at 43.688 105.918 90)
-			(effects
-				(font
-					(size 1.27 1.27)
-				)
-			)
-		)
-		(property "Footprint" ""
+			(at 46.228 103.886 90)
+			(effects
+				(font
+					(size 1.27 1.27)
+				)
+			)
+		)
+		(property "Value" "SW_Push_RightAngle"
+			(at 38.608 105.664 90)
+			(effects
+				(font
+					(size 1.27 1.27)
+				)
+			)
+		)
+		(property "Footprint" "tat_footprints:SW_Push_SHOU_HAN_SPST_RightAngle_TS24CA"
 			(at 46.99 105.41 0)
 			(effects
@@
 		(dnp no)
 		(property "Reference" "SW4"
-			(at 43.688 64.516 90)
-			(effects
-				(font
-					(size 1.27 1.27)
-				)
-			)
-		)
-		(property "Value" "SW_Push"
-			(at 43.688 66.548 90)
-			(effects
-				(font
-					(size 1.27 1.27)
-				)
-			)
-		)
-		(property "Footprint" ""
+			(at 46.228 64.516 90)
+			(effects
+				(font
+					(size 1.27 1.27)
+				)
+			)
+		)
+		(property "Value" "SW_Push_RightAngle"
+			(at 38.608 66.294 90)
+			(effects
+				(font
+					(size 1.27 1.27)
+				)
+			)
+		)
+		(property "Footprint" "tat_footprints:SW_Push_SHOU_HAN_SPST_RightAngle_TS24CA"
 			(at 46.99 66.04 0)
 			(effects
@@
 			)
 		)
-		(property "Description" "Push button switch, generic, two pins"
+		(property "Description" "TS24CA surface mount right angle switch"
 			(at 52.07 66.04 0)
 			(effects
@@
 		(on_board yes)
 		(dnp no)
-		(property "Reference" "R19"
+		(property "Reference" "R22"
 			(at 57.15 91.948 90)
 			(effects
@@
 			(project "tat_v1"
 				(path "/b6d2ddf1-6792-45dd-afc9-29fd74d587ec/c7fedf3e-0076-4d27-8f18-2fdc24044d55"
-					(reference "R19")
+					(reference "R22")
 					(unit 1)
 				)
@@
 		(dnp no)
 		(fields_autoplaced yes)
-		(property "Reference" "R23"
+		(property "Reference" "R26"
 			(at 67.31 130.8099 0)
 			(effects
@@
 			(project "tat_v1"
 				(path "/b6d2ddf1-6792-45dd-afc9-29fd74d587ec/c7fedf3e-0076-4d27-8f18-2fdc24044d55"
-					(reference "R23")
+					(reference "R26")
 					(unit 1)
 				)
@@
 			)
 		)
-		(property "Footprint" ""
+		(property "Footprint" "Sensor_Humidity:Sensirion_DFN-4_1.5x1.5mm_P0.8mm_SHT4x_NoCentralPad"
 			(at 161.29 91.44 0)
 			(effects
@@
 		(on_board yes)
 		(dnp no)
-		(property "Reference" "R20"
+		(property "Reference" "R23"
 			(at 57.15 132.588 90)
 			(effects
@@
 			(project "tat_v1"
 				(path "/b6d2ddf1-6792-45dd-afc9-29fd74d587ec/c7fedf3e-0076-4d27-8f18-2fdc24044d55"
-					(reference "R20")
+					(reference "R23")
 					(unit 1)
 				)
@@
 			)
 		)
-		(property "Footprint" ""
+		(property "Footprint" "Sensor_Humidity:Sensirion_DFN-4_1.5x1.5mm_P0.8mm_SHT4x_NoCentralPad"
 			(at 161.29 127 0)
 			(effects
@@
 		(dnp no)
 		(fields_autoplaced yes)
-		(property "Reference" "R26"
+		(property "Reference" "R29"
 			(at 245.11 88.8999 0)
 			(effects
@@
 			(project "tat_v1"
 				(path "/b6d2ddf1-6792-45dd-afc9-29fd74d587ec/c7fedf3e-0076-4d27-8f18-2fdc24044d55"
-					(reference "R26")
+					(reference "R29")
 					(unit 1)
 				)
@@
 		(dnp no)
 		(property "Reference" "SW6"
-			(at 43.688 144.526 90)
-			(effects
-				(font
-					(size 1.27 1.27)
-				)
-			)
-		)
-		(property "Value" "SW_Push"
-			(at 43.688 146.558 90)
-			(effects
-				(font
-					(size 1.27 1.27)
-				)
-			)
-		)
-		(property "Footprint" ""
+			(at 46.228 144.526 90)
+			(effects
+				(font
+					(size 1.27 1.27)
+				)
+			)
+		)
+		(property "Value" "SW_Push_RightAngle"
+			(at 38.608 146.304 90)
+			(effects
+				(font
+					(size 1.27 1.27)
+				)
+			)
+		)
+		(property "Footprint" "tat_footprints:SW_Push_SHOU_HAN_SPST_RightAngle_TS24CA"
 			(at 46.99 146.05 0)
 			(effects
@@
 		(dnp no)
 		(fields_autoplaced yes)
-		(property "Reference" "R27"
+		(property "Reference" "R30"
 			(at 254 88.8999 0)
 			(effects
@@
 			(project "tat_v1"
 				(path "/b6d2ddf1-6792-45dd-afc9-29fd74d587ec/c7fedf3e-0076-4d27-8f18-2fdc24044d55"
-					(reference "R27")
+					(reference "R30")
 					(unit 1)
 				)
@@
 		(dnp no)
 		(fields_autoplaced yes)
-		(property "Reference" "R24"
+		(property "Reference" "R27"
 			(at 137.16 82.5499 0)
 			(effects
@@
 			(project "tat_v1"
 				(path "/b6d2ddf1-6792-45dd-afc9-29fd74d587ec/c7fedf3e-0076-4d27-8f18-2fdc24044d55"
-					(reference "R24")
+					(reference "R27")
 					(unit 1)
 				)
@@
 		(on_board yes)
 		(dnp no)
-		(property "Reference" "R18"
+		(property "Reference" "R21"
 			(at 57.15 52.578 90)
 			(effects
@@
 			(project "tat_v1"
 				(path "/b6d2ddf1-6792-45dd-afc9-29fd74d587ec/c7fedf3e-0076-4d27-8f18-2fdc24044d55"
-					(reference "R18")
+					(reference "R21")
 					(unit 1)
 				)
@@
 		(dnp no)
 		(fields_autoplaced yes)
-		(property "Reference" "R21"
+		(property "Reference" "R24"
 			(at 67.31 50.7999 0)
 			(effects
@@
 			(project "tat_v1"
 				(path "/b6d2ddf1-6792-45dd-afc9-29fd74d587ec/c7fedf3e-0076-4d27-8f18-2fdc24044d55"
-					(reference "R21")
+					(reference "R24")
 					(unit 1)
 				)
@@
 		(dnp no)
 		(fields_autoplaced yes)
-		(property "Reference" "R22"
+		(property "Reference" "R25"
 			(at 67.31 90.1699 0)
 			(effects
@@
 			(project "tat_v1"
 				(path "/b6d2ddf1-6792-45dd-afc9-29fd74d587ec/c7fedf3e-0076-4d27-8f18-2fdc24044d55"
-					(reference "R22")
-					(unit 1)
-				)
+					(reference "R25")
+					(unit 1)
+				)
