File: hardware/schematic/tat_v1/peripherals.kicad_sch (KiCad schematic)
At the start: 21 parts, among them SW4 SW_Push_RightAngle, SW5 SW_Push_RightAngle, SW6 SW_Push_RightAngle, U5 STS4x, U6 SHT4x, U7 BL24C08F

Commit message: Fixed all footprint-symbol mismatches, ready to start routing!
Parts:
- SW4: symbol Switch:SW_Push -> tat_library:TS24CA
- SW5, SW6: symbol Switch:SW_Push -> tat_library:TS24CA; Link (none) -> https://www.lcsc.com/product-detail/Tactile-Switches_SHOU-H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
- U7: footprint Package_DFN_QFN:DFN-8-1EP_3x2mm_P0.5mm_EP1.3x1.5mm -> tat_footprints:EEPROM_BL24C08F-NTRC; Link (none) -> https://www.lcsc.com/product-detail/EEPROM_BL-Shanghai-Bell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
Changed lines of the file:
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@@
 			)
 		)
-		(property "Footprint" "Package_DFN_QFN:DFN-8-1EP_3x2mm_P0.5mm_EP1.3x1.5mm"
+		(property "Footprint" "tat_footprints:EEPROM_BL24C08F-NTRC"
 			(at 228.6 99.06 0)
 			(effects
@@
 			)
 		)
-		(property "Datasheet" ""
+		(property "Datasheet" "https://www.lcsc.com/datasheet/lcsc_datasheet_2410121550_BL-Shanghai-Belling-BL24C08F-NTRC_C5185882.pdf"
 			(at 228.6 99.06 0)
 			(effects
@@
 			)
 		)
+		(property "Link" "https://www.lcsc.com/product-detail/EEPROM_BL-Shanghai-Belling-BL24C08F-NTRC_C5185882.html?s_z=n_BL24C08F-NTRC"
+			(at 228.6 99.06 0)
+			(effects
+				(font
+					(size 1.27 1.27)
+				)
+				(hide yes)
+			)
+		)
 		(pin "3"
 		)
@@
 		(pin "7"
 		)
+		(pin "2"
+		)
+		(pin "1"
+		)
 		(instances
 			(project "tat_v1"
@@
 	)
 	(symbol
-		(lib_id "Switch:SW_Push")
+		(lib_id "tat_library:TS24CA")
 		(at 52.07 105.41 90)
 		(unit 1)
@@
 			)
 		)
-		(property "Datasheet" "~"
+		(property "Datasheet" "https://www.lcsc.com/datasheet/lcsc_datasheet_2404241539_SHOU-HAN-TS24CA_C393942.pdf"
 			(at 46.99 105.41 0)
 			(effects
@@
 			)
 		)
+		(property "Link" "https://www.lcsc.com/product-detail/Tactile-Switches_SHOU-HAN-TS24CA_C393942.html?s_z=n_SHOU%2520HAN%2520TS24CA"
+			(at 52.07 105.41 0)
+			(effects
+				(font
+					(size 1.27 1.27)
+				)
+				(hide yes)
+			)
+		)
 		(pin "2"
 		)
 		(pin "1"
 		)
+		(pin "3"
+		)
+		(pin "4"
+		)
 		(instances
 			(project "tat_v1"
@@
 	)
 	(symbol
-		(lib_id "Switch:SW_Push")
+		(lib_id "tat_library:TS24CA")
 		(at 52.07 66.04 90)
 		(unit 1)
@@
 			)
 		)
-		(property "Description" "TS24CA surface mount right angle switch"
+		(property "Description" "Push button switch, generic, two pins"
 			(at 52.07 66.04 0)
 			(effects
@@
 		)
 		(property "Link" "https://www.lcsc.com/product-detail/Tactile-Switches_SHOU-HAN-TS24CA_C393942.html?s_z=n_SHOU%2520HAN%2520TS24CA"
-			(at 52.07 66.04 90)
+			(at 52.07 66.04 0)
 			(effects
 				(font
@@
 		)
 		(pin "1"
+		)
+		(pin "4"
+		)
+		(pin "3"
 		)
 		(instances
@@
 	)
 	(symbol
-		(lib_id "Switch:SW_Push")
+		(lib_id "tat_library:TS24CA")
 		(at 52.07 146.05 90)
 		(unit 1)
@@
 			)
 		)
-		(property "Datasheet" "~"
+		(property "Datasheet" "https://www.lcsc.com/datasheet/lcsc_datasheet_2404241539_SHOU-HAN-TS24CA_C393942.pdf"
 			(at 46.99 146.05 0)
 			(effects
@@
 			)
 		)
+		(property "Link" "https://www.lcsc.com/product-detail/Tactile-Switches_SHOU-HAN-TS24CA_C393942.html?s_z=n_SHOU%2520HAN%2520TS24CA"
+			(at 52.07 146.05 0)
+			(effects
+				(font
+					(size 1.27 1.27)
+				)
+				(hide yes)
+			)
+		)
 		(pin "2"
 		)
 		(pin "1"
 		)
-		(instances
+		(pin "4"
+		)
+		(pin "3"
+		)
+		(instances
